File: PCBs/Expansion Board/Expansion Board.kicad_sch (KiCad schematic)
At the start: 6 parts, among them J1 Conn_02x08_Odd_Even, J2 Conn_02x08_Odd_Even, J3 Conn_02x05_Odd_Even, J4 Conn_02x05_Odd_Even

Commit message: Fixed some PCB stuff and rendering
Other:
- note added: "?"
- note added: "DISPLAY_SCL"
- note added: "DISPLAY_SDA"
- note added: "ROT_SW"
- note added: "SD_DETECT"
- note added: "SD_MISO"
- note added: "SD_MOSI"
- note added: "SD_SCK"
- note added: "SD_SS"
- note added: "S_E1"
- note added: "S_E2"
- moved on the sheet: J3, J4
