File: PCBs/Printer Mainboard/Printer Mainboard.kicad_pcb (KiCad board)
At the start: 4 copper layers, 110 x 175 mm, 280 parts, among them IC1 LM76005RNPR, J1 USB_A, J10 Conn_01x02, J11 Conn_02x08_Odd_Even, J12 Conn_02x08_Odd_Even, J13 Conn_01x04, J14 Conn_01x04, J15 Conn_01x04, J16 Conn_01x03, J17 Conn_01x03, J18 Conn_01x03, J19 Conn_01x03, J2 USB_C_Receptacle_USB2.0_14P, J20 Faston, J21 Faston, J22 Mini-DIN-4, J23 Conn_01x02, J24 Conn_01x02, J25 Conn_01x02, J26 Conn_01x04, J27 Conn_01x04, J28 Conn_01x04, J29 Conn_01x04, J3 Conn_01x02, J30 Conn_01x04, J31 Conn_01x06_Pin, J32 Conn_01x03, J33 Conn_01x02, J34 Conn_01x02, J35 Conn_01x03, J36 Conn_01x02, J37 Conn_01x02, J38 Conn_01x03, J39 Conn_01x02, J4 Conn_01x02, J40 Conn_01x02, J5 Conn_01x02, J6 Conn_01x02, J7 Conn_01x02, J8 Conn_01x02, J9 Conn_01x02, K1 G2RL-1A-E, Q1 NVMFWS4D5N08XT1G, Q2 NVMFWS4D5N08XT1G, Q3 NVMFWS4D5N08XT1G, Q4 NVMFWS4D5N08XT1G, Q5 BC817, Q6 BC817, Q7 BC817, Q8 BC817, Q9 BC807, SW1 SW_SPST, SW2 SW_Push, SW3 SW_Push, U1 USBLC6-2SC6, U10 TMC2130-TA, U11 TMC2130-TA, U12 STM32H743VITx, U2 AP7361C-33E, U3 TC4427xOA, U4 TC4427xOA, U5 SN74LV4T125, U6 NE555D, U7 TMC2130-TA, U8 TMC2130-TA, U9 TMC2130-TA, Y1 25MHz

Commit message: Fixed some PCB stuff and rendering
Parts:
- added G***: LOGO, Art:Scorpion drawing, F.Cu at (62.3, 47.1)
- added G***: LOGO, Art:Scorpion drawing, F.Cu at (84.2, 123.2)
- added G***: LOGO, Art:Scorpion drawing, F.Cu at (127.6, 149.7)
- added G***: LOGO, Art:Scorpion drawing, F.Cu at (120.0, 89.9)
- added G***: LOGO, Art:Scorpion drawing, F.Cu at (120.2, 45.9)
- added G***: LOGO, Art:RAWR, B.Cu at (68.6, 121.5)
Other:
- board text added: "3.3V"
- board text added: "5 euro? op je muil, gauw!"
- board text added: "5V"
- board text added: ":)"
- board text added: "BOOT"
- board text added: "Expansion slot"
- board text added: "FAN"
- board text added: "FAN 1"
- board text added: "FAN 2"
- board text added: "FAN 3"
- board text added: "FAN 4"
- board text added: "FAN POWER SELECT"
- board text added: "GND"
- board text added: "LIM 1"
- board text added: "LIM 2"
- board text added: "LIM 3"
- board text added: "LIM 4"
- board text added: "MOT 1"
- board text added: "MOT 2"
- board text added: "MOT 3"
- board text added: "MOT 4"
- board text added: "MOT 5"
- board text added: "RESET"
- board text added: "SWD_CLK"
- board text added: "SWD_DIO"
- board text added: "Safety"
- board text added: "Safety Reset"
- board text added: "TEMP Module"
- board text added: "Ther 1"
- board text added: "Ther 2"
- board text added: "Ther 3"
- board text added: "VS"
- board text added: "Very expensive :)"
- board text added: "by looking at this you have voided the warranty"
